Commit message: fix: visual correctness

File: uav_gazebo/urdf/example_ruckig_position.xacro (robot description, xacro)
@@ -39,5 +39,5 @@
   <link name="link1">
     <inertial>
-      <origin xyz="0 ${link_length1/2} 0" rpy="0 0 0"/>
+      <origin xyz="0 ${link_length1/2} 0" rpy="1.5708 0 0"/>
       <mass    value="${mass1}"/>
       <inertia
@@ -46,5 +46,5 @@
     </inertial>
     <visual>
-      <origin xyz="0 ${link_length1/2} 0" rpy="0 0 0"/>
+      <origin xyz="0 ${link_length1/2} 0" rpy="1.5708 0 0"/>
       <geometry>
         <cylinder radius="${link_radius}" length="${link_length1}"/>
@@ -58,5 +58,5 @@
   <link name="link2">
     <inertial>
-      <origin xyz="0 ${link_length2/2} 0" rpy="0 0 0"/>
+      <origin xyz="0 ${link_length2/2} 0" rpy="1.5708 0 0"/>
       <mass    value="${mass2}"/>
       <inertia
@@ -65,5 +65,5 @@
     </inertial>
     <visual>
-      <origin xyz="0 ${link_length2/2} 0" rpy="0 0 0"/>
+      <origin xyz="0 ${link_length2/2} 0" rpy="1.5708 0 0"/>
       <geometry>
         <cylinder radius="${link_radius}" length="${link_length2}"/>
@@ -77,5 +77,5 @@
   <link name="link3">
     <inertial>
-      <origin xyz="0 ${link_length3/2} 0" rpy="0 0 0"/>
+      <origin xyz="0 ${link_length3/2} 0" rpy="1.5708 0 0"/>
       <mass    value="${mass3}"/>
       <inertia
@@ -84,5 +84,5 @@
     </inertial>
     <visual>
-      <origin xyz="0 ${link_length3/2} 0" rpy="0 0 0"/>
+      <origin xyz="0 ${link_length3/2} 0" rpy="1.5708 0 0"/>
       <geometry>
         <cylinder radius="${link_radius}" length="${link_length3}"/>
